Commit message: done

File: body.urdf (robot description, URDF)
Before this commit: robot robot, 1 links, 0 joints
Links:
- added link Link2, mass 1; collision box size=0.3267144362080938 0.0725489880034792 0.4276493913060828; visual box size=0.3267144362080938 0.0725489880034792 0.4276493913060828
- link Link1: geometry collision box size=0.221409318973732 0.03321225170151271 0.38014502805940537; visual box size=0.221409318973732 0.03321225170151271 0.38014502805940537
Joints:
- added joint Link1_Link2: type revolute, parent Link1, child Link2, origin xyz=0.110704659486866 0 0.38014502805940537 rpy=0 0 0, axis 0 1 0, limit lower=-3.14159 upper=3.14159 effort=0.0 velocity=0.0

Commit message: done

File: body.urdf (robot description, URDF)
Before this commit: robot robot, 2 links, 1 joints
Links:
- added link Link3, mass 1; collision box size=0.18871405631231997 0.29145477249192236 0.12759028221349816; visual box size=0.18871405631231997 0.29145477249192236 0.12759028221349816
- added link Link4, mass 1; collision box size=0.4558763822671102 0.21825181291179213 0.29963039541311554; visual box size=0.4558763822671102 0.21825181291179213 0.29963039541311554
- added link Link5, mass 1; collision box size=0.07733837970252738 0.26056760554640945 0.12972691509796813; visual box size=0.07733837970252738 0.26056760554640945 0.12972691509796813
- added link Link6, mass 1; collision box size=0.05668253274871987 0.1437955046651676 0.048896376470993264; visual box size=0.05668253274871987 0.1437955046651676 0.048896376470993264
- link Link1: geometry collision box size=0.06608473046792523 0.020500609180380436 0.3190513140909531; visual box size=0.06608473046792523 0.020500609180380436 0.3190513140909531
- link Link2: geometry collision box size=0.42384011714147785 0.2353823488694477 0.13592080034438836; visual box size=0.42384011714147785 0.2353823488694477 0.13592080034438836
Joints:
- added joint Link2_Link3: type revolute, parent Link2, child Link3, origin xyz=0.42384011714147785 0 0.13592080034438836 rpy=0 0 0, axis 0 1 0, limit lower=-3.14159 upper=3.14159 effort=0.0 velocity=0.0
- added joint Link3_Link4: type revolute, parent Link3, child Link4, origin xyz=0.18871405631231997 0 0.12759028221349816 rpy=0 0 0, axis 0 1 0, limit lower=-3.14159 upper=3.14159 effort=0.0 velocity=0.0
- added joint Link4_Link5: type revolute, parent Link4, child Link5, origin xyz=0.4558763822671102 0 0.29963039541311554 rpy=0 0 0, axis 0 1 0, limit lower=-3.14159 upper=3.14159 effort=0.0 velocity=0.0
- added joint Link5_Link6: type revolute, parent Link5, child Link6, origin xyz=0.07733837970252738 0 0.12972691509796813 rpy=0 0 0, axis 0 1 0, limit lower=-3.14159 upper=3.14159 effort=0.0 velocity=0.0
- joint Link1_Link2: origin xyz=0.110704659486866 0 0.38014502805940537 rpy=0 0 0 -> xyz=0.03304236523396262 0 0.3190513140909531 rpy=0 0 0
